File: RP_12MHz_crystal.kicad_sch (KiCad schematic)
At the start: 0 parts

Commit message: Downloaded the Footprints for RP2350B
Downloaded the ABM8-272-T3 for the crystal and the SM03B-SRSS-TB for the JST connector, though the later is not correct (I think) because it lacks mechanical pads within the footprint.
Parts:
- added C3, C4: 15p, symbol Device:C
- added R2: 1k, symbol Device:R
- added X1: ABM8-272-T3, ABM8-272-T3_ABR, symbol ABM8-272-T3:ABM8-272-T3
Connections:
- new net: C3.2, R2.2, X1.3
- new net GND: C3.1, C4.2, X1.2, X1.4
- new net XIN: C4.1, X1.1
- new net XOUT: R2.1
