File: ACS.kicad_sch (KiCad schematic)
At the start: 0 parts

Commit message: Update
Parts:
- added C36, C38: 22uF, Capacitor_SMD:C_0805_2012Metric, symbol Device:C
- added C37, C39, C44: 2.2uF, Capacitor_SMD:C_0603_1608Metric, symbol Device:C
- added C40, C41, C42, C43, C45, C46, C47, C49: 100nF, Capacitor_SMD:C_0603_1608Metric, symbol Device:C
- added C48: 1.0uF, Capacitor_SMD:C_0603_1608Metric, symbol Device:C
- added C50: 22nF, Capacitor_SMD:C_0603_1608Metric, symbol Device:C
- added D10, D11, D8, D9: MMBZ15VALT1G, Package_TO_SOT_SMD:SOT-23, symbol Device:D_Zener_Dual_CommonAnode_KKA
- added Q5, Q7: PMBT2222A, Package_TO_SOT_SMD:SOT-23, symbol Transistor_BJT:PMBT2222A
- added Q6: IRF9393, Package_SO:SOIC-8_3.9x4.9mm_P1.27mm, symbol Transistor_FET:IRF7404
- added R47: 200m 1W, Resistor_SMD:R_2010_5025Metric, symbol Device:R_US
- added R54: 15k, Resistor_SMD:R_0603_1608Metric, symbol Device:R_US
- added RN8, RN9: 4.7k, Resistor_SMD:R_Array_Convex_4x0603, symbol Device:R_Pack04_Split
- added U2: BMX160, Package_LGA:Bosch_LGA-14_3x2.5mm_P0.5mm, symbol Sensor_Motion:BMI160
- added U8: KF33BDT, Package_TO_SOT_SMD:TO-252-2, symbol Regulator_Linear:KF33BDT
- added U9: MAX22200, Package_DFN_QFN:QFN-32-1EP_5x5mm_P0.5mm_EP3.1x3.1mm_ThermalVias, symbol nyansat-symbols:MAX22200
Connections:
- new net: R54.1, U9.18 (IREF)
- new net: RN8.4 (R4.1), U9.1 (~{FAULT})
- new net: Q5.3 (C), RN9.3 (R3.1), RN9.4 (R4.1)
- new net: C37.2, Q6.4 (G), RN9.5 (R4.2)
- new net: Q5.1 (B), RN9.7 (R2.2), RN9.8 (R1.2)
- new net: C44.1, U9.20 (V_{18})
- new net: C50.2, U9.22 (C_{FN})
- new net: C50.1, U9.23 (C_{FP})
- new net: C48.2, U9.24 (V_{CP})
- new net: Q6.1 (S), Q6.2 (S), Q6.3 (S), R47.2
- new net FBRDG3V3: C45.1, C46.1, C47.1, C49.1, RN8.5 (R4.2), RN8.6 (R3.2), RN8.7 (R2.2), U8.3 (VO)
- new net FBRGEN: Q7.3 (C), RN8.2 (R2.1), U9.21 (ENABLE)
- new net GND: C36.1, C38.2, C39.2, C40.2, C41.2, C42.2, C43.2, C44.2, C45.2, C46.2, C47.2, C49.2, D10.3 (A), D11.3 (A), D8.3 (A), D9.3 (A), Q5.2 (E), Q7.2 (E), R54.2, RN9.2 (R2.1), U8.2 (GND), U9.17 (TRIGB), U9.19 (GND), U9.33 (PAD), U9.4 (GND), U9.8 (TRIGA)
- new net MISO: RN8.3 (R3.1), U9.7 (SDO)
- new net OUT1A: D8.1 (K), U9.31 (OUT0)
- new net OUT1B: D8.2 (K), U9.30 (OUT1)
- new net OUT2A: D9.1 (K), U9.27 (OUT2)
- new net OUT2B: D9.2 (K), U9.26 (OUT3)
- new net OUT3A: D10.1 (K), U9.10 (OUT4)
- new net OUT3B: D10.2 (K), U9.11 (OUT5)
- new net OUT4A: D11.2 (K), U9.14 (OUT6)
- new net OUT4B: D11.1 (K), U9.15 (OUT7)
- new net PWREN: RN9.1 (R1.1)
- new net RAWPWR: C36.2, C37.1, R47.1, RN9.6 (R3.2)
- new net VM: C38.1, C39.1, C40.1, C41.1, C42.1, C43.1, C48.1, Q6.5 (D), Q6.6 (D), Q6.7 (D), Q6.8 (D), U8.1 (VI), U9.12 (V_{M}), U9.13 (V_{M}), U9.16 (V_{M}), U9.25 (V_{M}), U9.28 (V_{M}), U9.29 (V_{M}), U9.32 (V_{M}), U9.9 (V_{M})
Other:
- note added: "Is there any reason for having a seperate regulator?"
- note added: "Linearize power switch to limit inrush; limit fault currents."
- note added: "Threshold ~3A/V; dv/dt through thresh 591uV/us dA/dt 1.8mA/us peaks at around 800mA"
