File: RP_primary_flash.kicad_sch (KiCad schematic)
At the start: 5 parts, among them U5 W25Q128JVS

Commit message: Consolidate/mostly finalize avionics
Add RP2350 components to same sheet as RP2350, replace flash with MRAM
Parts:
- removed C2: 100n, symbol Device:C
- removed R1, R9: DNF, symbol Device:R
- removed R10: 0, symbol Device:R
- removed U5: W25Q128JVS, Package_SO:SOIC-8_5.3x5.3mm_P1.27mm, symbol Memory_Flash:W25Q128JVS
Other:
- note removed: "Why are there resistors with R = 0 or DNF???"
