File: RP_secondary_flash_psram.kicad_sch (KiCad schematic)
At the start: 4 parts, among them U6 W25Q128JVS

Commit message: Consolidate/mostly finalize avionics
Add RP2350 components to same sheet as RP2350, replace flash with MRAM
Parts:
- removed C22: DNF, symbol Device:C
- removed R11, R13: DNF, symbol Device:R
- removed U6: W25Q128JVS, Package_SO:SOIC-8_5.3x5.3mm_P1.27mm, symbol Memory_Flash:W25Q128JVS
Other:
- note removed: "Optional Secondary flash or PSRAM (U4), using the second chip select (XIP_SS_N[1]) on GPIO0. N.B. Pull-up R13 will be required as GPIOs default to pull-downs at power-up."
- note removed: "Why are there resistors with R = DNF???"
