File: owlsat.kicad_sch (KiCad schematic)
At the start: 0 parts

Commit message: Update
Other:
- sheet Burn Wires renamed Burn Wires and Thermal
- note added: "OwlSat was developed by students at Rice University under the direction of Dr. Patricia Reiff, Charlotte, Brandon, Luke, Roman, Enzo, Andrew, Clay, Jose... Based off the Obi Wan Komputer based on the work of students at Oakwood High School under the direction of Michael Lyle In turn based on the PyCubed project by Maximilian Holliday As all previous work was licensed under CC BY-SA 4.0, this work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"
- note removed: "OwlSat was developed by students at Rice University under the direction of Dr. Patricia Reiff, Charlotte, Luke, Roman, Enzo... Based off the Obi Wan Komputer based on the work of students at Oakwood High School under the direction of Michael Lyle In turn based on the PyCubed project by Maximilian Holliday As all previous work was licensed under CC BY-SA 4.0, this work OwlSat Mainboard (c) 2025- b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"
Changed lines of the file:
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@@
 		)
 	)
-	(text "OwlSat was developed by students at Rice University\nunder the direction of Dr. Patricia Reiff, Charlotte, \nLuke, Roman, Enzo...\nBased off the Obi Wan Komputer based on the work of \nstudents at Oakwood High School under the direction of Michael Lyle\nIn turn based on the PyCubed project by Maximilian Holliday\n\nAs all previous work was licensed under CC BY-SA 4.0,\nthis work OwlSat Mainboard (c) 2025- by Rice University\nis licensed under the same license. To view a copy of this license, visit\nhttps://creativecommons.org/licenses/by-sa/4.0/"
+	(text "OwlSat was developed by students at Rice University\nunder the direction of Dr. Patricia Reiff, Charlotte, \nBrandon, Luke, Roman, Enzo, Andrew, Clay, Jose...\nBased off the Obi Wan Komputer based on the work of \nstudents at Oakwood High School under the direction of Michael Lyle\nIn turn based on the PyCubed project by Maximilian Holliday\n\nAs all previous work was licensed under CC BY-SA 4.0,\nthis work OwlSat Mainboard (c) 2025- by Rice University\nis licensed under the same license. To view a copy of this license, visit\nhttps://creativecommons.org/licenses/by-sa/4.0/"
 		(exclude_from_sim no)
 		(at 14.732 26.416 0)
@@
 			(color 0 0 0 0.0000)
 		)
-		(property "Sheetname" "Burn Wires"
+		(property "Sheetname" "Burn Wires and Thermal"
 			(at 110.49 48.8184 0)
 			(effects
